File: luzNocturna.kicad_pcb (KiCad board)
At the start: 2 copper layers, 52 x 52 mm, 18 parts, among them J1 CON, Q1 2N3904BU, U1 TL082, U2 SRD-XXVDC

Commit message: agregando logo
Parts:
- added G***: LOGO, MSS_Devices:logo-mr, B.Cu at (143.7, 78.7)
- added G***: LOGO, MSS_Devices:logo-mr_78x3.6mm, F.Cu at (152.8, 115.8)

Commit message: actualizando a version 7, aun no se pueden ver los modelos 3D
Parts:
- U2: value SRD-XXVDC -> SANYOU_SRD_Form_C
Connections:
- J1 pad 1: (no net) -> /fuente-sin-transformador/SW
- U2 pad 3: (no net) -> /SW
- U2 pad 4: (no net) -> unconnected-(U2-Pad4)
Other:
- net class Default removed
